File: PCB/BlinkerLED.kicad_pcb (KiCad board)
At the start: 2 copper layers, 99.1 x 99.1 mm, 19 parts, among them J1 Conn_01x02_Socket, J2 Conn_01x01_Socket, U1 NE555P, U2 4017

Commit message: Add files via upload
Parts:
- moved C3 51.2 mm to (117.5, 130.5), turned to 180 degrees
- moved C4 27.2 mm to (103.0, 129.0)
- moved R4 12.8 mm to (130.3, 136.5), turned to 180 degrees
- moved J1 4.44 mm to (120.5, 142.5), turned to 0 degrees
- moved D5 3.84 mm to (138.8, 130.0), turned to 180 degrees
- moved D2 2.54 mm to (138.3, 73.5), turned to 180 degrees
- moved J2 2.50 mm to (101.0, 121.5)
- moved D3 2.31 mm to (148.8, 91.5), turned to 180 degrees
- moved D4 2.27 mm to (148.5, 112.0), turned to 180 degrees
- moved D6 1.97 mm to (109.5, 141.8), turned to 90 degrees
- moved D1 1.49 mm to (109.0, 60.7), turned to -90 degrees
Routing:
- net GND: track 164.2 -> 92.2 mm
- net Net-(U1-CONT): track 53.3 -> 6.82 mm
- net Net-(D8-A): track 35.2 -> 65.7 mm
- net Net-(D9-A): track 88.4 -> 58.1 mm
- net Net-(D7-A): track 38.0 -> 67.2 mm
- net Net-(D3-A): track 100.3 -> 76.3 mm
- net Net-(D5-A): track 40.8 -> 60.7 mm
- net Net-(D10-A): track 59.2 -> 77.0 mm
- net +5V: track 78.0 -> 93.3 mm
- net OUT: track 82.9 -> 68.0 mm
- net TR: track 41.0 -> 54.0 mm
- net Net-(D2-A): track 48.1 -> 61.1 mm
- net Net-(U1-DISCH): track 56.6 -> 44.7 mm
- net Net-(D4-A): track 94.4 -> 103.5 mm
- net Net-(D6-A): track 52.6 -> 56.9 mm
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
Commit message: Add files via upload
Parts:
- moved RV1 38.8 mm to (99.0, 135.5)
Routing:
- net Net-(D3-A): track 76.3 -> 47.0 mm
- net Net-(U1-DISCH): track 44.7 -> 60.5 mm
- net TR: track 54.0 -> 58.9 mm
Changed lines of the file:
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@@
 	(footprint "Potentiometer_THT:Potentiometer_Vishay_T93YA_Vertical"
 		(layer "F.Cu")
-		(at 93.46 97.1125)
+		(at 98.96 135.5)
 		(descr "Potentiometer, vertical, Vishay, https://www.vishay.com/docs/51026/t93.pdf")
 		(tags "Potentiometer vertical vishay")
@@
 		)
 		(embedded_fonts no)
+		(model "C:/Users/sabom/Desktop/BlinkerLED/ul_CD4017BE/KiCADv6/footprints.pretty/N16.kicad_mod"
+			(offset
+				(xyz 0 0 0)
+			)
+			(scale
+				(xyz 1 1 1)
+			)
+			(rotate
+				(xyz 0 0 0)
+			)
+		)
 	)
 	(footprint "Capacitor_THT:C_Disc_D7.5mm_W2.5mm_P5.00mm"
@@
 	)
 	(segment
-		(start 106.296 115.296)
-		(end 106.296 117.629)
+		(start 99.448 130.908)
+		(end 99.448 120.05084)
 		(width 0.2)
 		(layer "F.Cu")
@@
 	)
 	(segment
+		(start 104.04 135.5)
+		(end 99.448 130.908)
+		(width 0.2)
+		(layer "F.Cu")
+		(net 3)
+	)
+	(segment
+		(start 104.40984 115.089)
+		(end 105.98016 115.089)
+		(width 0.2)
+		(layer "F.Cu")
+		(net 3)
+	)
+	(segment
 		(start 105.044888 129)
 		(end 105.085 129)
@@
 	)
 	(segment
-		(start 104.73895 124.911)
-		(end 104.094 124.26605)
+		(start 105.98016 115.089)
+		(end 106.296 115.40484)
 		(width 0.2)
 		(layer "F.Cu")
@@
 	)
 	(segment
-		(start 106.296 117.629)
-		(end 105.195 118.73)
+		(start 104.73895 124.911)
+		(end 104.094 124.26605)
 		(width 0.2)
 		(layer "F.Cu")
@@
 	)
 	(segment
+		(start 106.296 115.40484)
+		(end 106.296 117.629)
+		(width 0.2)
+		(layer "F.Cu")
+		(net 3)
+	)
+	(segment
 		(start 109.174 124.911)
 		(end 104.73895 124.911)
@@
 	)
 	(segment
-		(start 105.085 129)
-		(end 112.815 121.27)
+		(start 99.448 120.05084)
+		(end 104.40984 115.089)
 		(width 0.2)
 		(layer "F.Cu")
@@
 	)
 	(segment
-		(start 98.54 107.54)
-		(end 106.296 115.296)
+		(start 106.296 117.629)
+		(end 105.195 118.73)
 		(width 0.2)
 		(layer "F.Cu")
@@
 	)
 	(segment
-		(start 104.094 124.26605)
-		(end 104.094 123.35395)
+		(start 105.085 129)
+		(end 112.815 121.27)
 		(width 0.2)
 		(layer "F.Cu")
@@
 	)
 	(segment
-		(start 98.54 97.1125)
-		(end 98.54 107.54)
+		(start 104.094 124.26605)
+		(end 104.094 123.35395)
 		(width 0.2)
 		(layer "F.Cu")
@@
 	)
 	(segment
-		(start 110.9087 93.5913)
-		(end 104.88 99.62)
+		(start 113.5 98.5)
+		(end 106 98.5)
 		(width 0.2)
 		(layer "F.Cu")
@@
 	)
 	(segment
-		(start 112.250365 93.5913)
-		(end 110.9087 93.5913)
+		(start 120.5 91.5)
+		(end 113.5 98.5)
 		(width 0.2)
 		(layer "F.Cu")
@@
 	)
 	(segment
-		(start 118.5 75.5)
-		(end 113.4487 70.4487)
-		(width 0.2)
-		(layer "F.Cu")
-		(net 7)
-	)
-	(segment
-		(start 113.4487 70.4487)
-		(end 113.4487 92.392965)
-		(width 0.2)
-		(layer "F.Cu")
-		(net 7)
-	)
-	(segment
-		(start 146.23 89.23)
-		(end 132.5 75.5)
+		(start 106 98.5)
+		(end 104.88 99.62)
 		(width 0.2)
 		(layer "F.Cu")
@@
 	)
 	(segment
-		(start 113.4487 92.392965)
-		(end 112.250365 93.5913)
+		(start 146.23 91.5)
+		(end 120.5 91.5)
 		(width 0.2)
 		(layer "F.Cu")
@@
 	)
 	(segment
-		(start 132.5 75.5)
-		(end 118.5 75.5)
-		(width 0.2)
-		(layer "F.Cu")
-		(net 7)
-	)
-	(segment
 		(start 105.272965 101.2113)
 		(end 104.487035 101.2113)
@@
 	)
 	(segment
-		(start 97.126 95.9865)
-		(end 99.006405 95.9865)
+		(start 104.24374 114.688)
+		(end 108.773 114.688)
 		(width 0.2)
 		(layer "F.Cu")
@@
 	)
 	(segment
-		(start 110.73 118.73)
-		(end 112.815 118.73)
+		(start 101.5 135.5)
+		(end 99.047 133.047)
 		(width 0.2)
 		(layer "F.Cu")
@@
 	)
 	(segment
-		(start 96 97.1125)
-		(end 93.46 97.1125)
+		(start 100.31 110.75426)
+		(end 104.24374 114.688)
 		(width 0.2)
 		(layer "F.Cu")
@@
 	)
 	(segment
-		(start 99.666 97.578905)
-		(end 99.5 97.744905)
+		(start 108.773 114.688)
+		(end 112.815 118.73)
 		(width 0.2)
 		(layer "F.Cu")
@@
 	(segment
 		(start 100.31 90)
-		(end 100.31 92.8025)
-		(width 0.2)
-		(layer "F.Cu")
-		(net 17)
-	)
-	(segment
-		(start 99.5 107.5)
-		(end 110.73 118.73)
-		(width 0.2)
-		(layer "F.Cu")
-		(net 17)
-	)
-	(segment
-		(start 99.5 97.744905)
-		(end 99.5 107.5)
-		(width 0.2)
-		(layer "F.Cu")
-		(net 17)
-	)
-	(segment
-		(start 99.006405 95.9865)
-		(end 99.666 96.646095)
-		(width 0.2)
-		(layer "F.Cu")
-		(net 17)
-	)
-	(segment
-		(start 100.31 92.8025)
-		(end 96 97.1125)
+		(end 100.31 110.75426)
 		(width 0.2)
 		(layer "F.Cu")
@@
 	)
 	(segment
-		(start 99.666 96.646095)
-		(end 99.666 97.578905)
+		(start 99.047 119.88474)
+		(end 104.24374 114.688)
 		(width 0.2)
 		(layer "F.Cu")
@@
 	)
 	(segment
-		(start 96 97.1125)
-		(end 97.126 95.9865)
+		(start 99.047 133.047)
+		(end 99.047 119.88474)
 		(width 0.2)
 		(layer "F.Cu")
